Commit message: Refactored codebase, that contains the full kinematic feasibility along with all RobotStudio tests like ik and fk parity tests

File: Assests/Robot APCC/IRB-1300-1400-URDF-New/urdf/IRB-1300-1400-URDF.urdf (robot description, URDF)
Before this commit: robot IRB-1300 1400 URDF, 7 links, 6 joints
Links:
- link Base: geometry collision mesh filename=../meshes/Base.STL; visual mesh filename=../meshes/Base.STL
- link Link_1: geometry collision mesh filename=../meshes/Link_1.STL; visual mesh filename=../meshes/Link_1.STL
- link Link_2: geometry collision mesh filename=../meshes/Link_2.STL; visual mesh filename=../meshes/Link_2.STL
- link Link_3: geometry collision mesh filename=../meshes/Link_3.STL; visual mesh filename=../meshes/Link_3.STL
- link Link_4: geometry collision mesh filename=../meshes/Link_4.STL; visual mesh filename=../meshes/Link_4.STL
- link Link_5: geometry collision mesh filename=../meshes/Link_5.STL; visual mesh filename=../meshes/Link_5.STL
- link Link_6: geometry collision mesh filename=../meshes/Link_7.STL; visual mesh filename=../meshes/Link_7.STL

File: Assests/Robot APCC/IRB-1300-1400-URDF-New/urdf/IRB-1300-1400-URDF_ee.urdf (robot description, URDF)
Before this commit: robot IRB-1300 1400 URDF, 7 links, 6 joints
Links:
- added link ee_link
- link Base: geometry collision mesh filename=../meshes/Base.STL; visual mesh filename=../meshes/Base.STL
- link Link_1: geometry collision mesh filename=../meshes/Link_1.STL; visual mesh filename=../meshes/Link_1.STL
- link Link_2: geometry collision mesh filename=../meshes/Link_2.STL; visual mesh filename=../meshes/Link_2.STL
- link Link_3: geometry collision mesh filename=../meshes/Link_3.STL; visual mesh filename=../meshes/Link_3.STL
- link Link_4: geometry collision mesh filename=../meshes/Link_4.STL; visual mesh filename=../meshes/Link_4.STL
- link Link_5: geometry collision mesh filename=../meshes/Link_5.STL; visual mesh filename=../meshes/Link_5.STL
- link Link_6: geometry collision mesh filename=../meshes/Link_7.STL; visual mesh filename=../meshes/Link_7.STL
Joints:
- added joint ee_joint: type fixed, parent Link_6, child ee_link, origin xyz=0.0998237 0.123033 0.0828027 rpy=0.001199 0.000599 2.782547
