Commit message: Changed link naming convention in urdf, then added correct urdf path names

File: Assests/Robot APCC/IRB-1300 1150 URDF/urdf/IRB 1300-1150 URDF_ee.urdf (robot description, URDF)
Before this commit: robot IRB 1300-1150 URDF, 8 links, 7 joints
Links:
- removed link Link1
- removed link Link2
- removed link Link3
- removed link Link4
- removed link Link5
- removed link Link6
- added link Link_1, mass 16.3325331099999; collision mesh filename=package://IRB 1300-1150 URDF/meshes/Link1.STL; visual mesh filename=package://IRB 1300-1150 URDF/meshes/Link1.STL
- added link Link_2, mass 15.4405289883218; collision mesh filename=package://IRB 1300-1150 URDF/meshes/Link2.STL; visual mesh filename=package://IRB 1300-1150 URDF/meshes/Link2.STL
- added link Link_3, mass 4.41745625966426; collision mesh filename=package://IRB 1300-1150 URDF/meshes/Link3.STL; visual mesh filename=package://IRB 1300-1150 URDF/meshes/Link3.STL
- added link Link_4, mass 3.69431402699864; collision mesh filename=package://IRB 1300-1150 URDF/meshes/Link4.STL; visual mesh filename=package://IRB 1300-1150 URDF/meshes/Link4.STL
- added link Link_5, mass 0.585190237279786; collision mesh filename=package://IRB 1300-1150 URDF/meshes/Link5.STL; visual mesh filename=package://IRB 1300-1150 URDF/meshes/Link5.STL
- added link Link_6, mass 0.00790032012561492; collision mesh filename=package://IRB 1300-1150 URDF/meshes/Link6.STL; visual mesh filename=package://IRB 1300-1150 URDF/meshes/Link6.STL
Joints:
- removed joint Joint1
- removed joint Joint2
- removed joint Joint3
- removed joint Joint4
- removed joint Joint5
- removed joint Joint6
- added joint Joint_1: type revolute, parent base_link, child Link_1, origin xyz=0 0 0.254 rpy=0 0 0, axis 0 0 1, limit lower=-3.1416 upper=3.1416 effort=1 velocity=1
- added joint Joint_2: type revolute, parent Link_1, child Link_2, origin xyz=0.15 0 0.29 rpy=0 0 0, axis 0 1 0, limit lower=-1.6581 upper=2.7053 effort=1 velocity=1
- added joint Joint_3: type revolute, parent Link_2, child Link_3, origin xyz=0 0 0.575 rpy=0 0 0, axis 0 1 0, limit lower=-3.6652 upper=1.1345 effort=1 velocity=1
- added joint Joint_4: type revolute, parent Link_3, child Link_4, origin xyz=0.128 0 0.04 rpy=0 0 0, axis 1 0 0, limit lower=-4.0143 upper=4.0143 effort=1 velocity=1
- added joint Joint_5: type revolute, parent Link_4, child Link_5, origin xyz=0.297 0 0 rpy=0 0 0, axis 0 1 0, limit lower=-2.2689 upper=2.2689 effort=1 velocity=1
- added joint Joint_6: type revolute, parent Link_5, child Link_6, origin xyz=0.0900000000000001 0 0 rpy=0 0 0, axis 1 0 0, limit lower=-4.2237 upper=4.2237 effort=1 velocity=1
- joint ee_joint: parent Link6 -> Link_6
