Commit message: updated URDF naming and file name conventions, made neccessary changes

File: Assests/Robot APCC/IRB_1300_1150_URDF/IRB-1300-1150 URDF_v2/urdf/IRB_1300_1150_URDF_with_fixture.urdf (robot description, URDF)
Before this commit: robot IRB-1300 900 URDF, 7 links, 6 joints
Links:
- removed link base_link
- added link Base_link, mass 13.1816717182696; collision mesh filename=../meshes/Base_link.STL; visual mesh filename=../meshes/Base_link.STL
- added link ee_link
- link Link_1: mass 15143711685.0337 -> 16.33253311; geometry collision mesh filename=../meshes/Link_1.STL; visual mesh filename=../meshes/Link_1.STL
- link Link_2: mass 13168240511.6789 -> 15.4405289883218; geometry collision mesh filename=../meshes/Link_2.STL; visual mesh filename=../meshes/Link_2.STL
- link Link_3: mass 4421135022.18643 -> 4.41745625966426; geometry collision mesh filename=../meshes/Link_3.STL; visual mesh filename=../meshes/Link_3.STL
- link Link_4: mass 3695342210.06587 -> 3.69431403174966; geometry collision mesh filename=../meshes/Link_4.STL; visual mesh filename=../meshes/Link_4.STL
- link Link_5: mass 586394466.626242 -> 0.585190237279786; geometry collision mesh filename=../meshes/Link_5.STL; visual mesh filename=../meshes/Link_5.STL
- link Link_6: mass 7900320.12561475 -> 0.00790032012561492; geometry collision mesh filename=../meshes/Link_6.STL; visual mesh filename=../meshes/Link_6.STL
Joints:
- added joint ee_joint: type fixed, parent Link_6, child ee_link, origin xyz=0.0998237 0.123033 0.0828027 rpy=0.001199 0.000599 2.782547
- joint Joint_1: limit lower=-3.142 upper=3.142 effort=1 velocity=1 -> lower=-3.1416 upper=3.1416 effort=1 velocity=1; parent base_link -> Base_link
- joint Joint_2: limit lower=-1.745 upper=2.269 effort=1 velocity=1 -> lower=-1.6581 upper=2.7053 effort=1 velocity=1; origin xyz=0.05 0 0.29 rpy=0 0 0 -> xyz=0.15 0 0.29 rpy=0 0 0
- joint Joint_3: limit lower=-3.665 upper=1.134 effort=1 velocity=1 -> lower=-3.6652 upper=1.1345 effort=1 velocity=1; origin xyz=0 0 0.425 rpy=0 0 0 -> xyz=0 0 0.575 rpy=0 0 0
- joint Joint_4: limit lower=-4.014 upper=4.014 effort=1 velocity=1 -> lower=-4.0143 upper=4.0143 effort=1 velocity=1; origin xyz=0.1295 0 0.04 rpy=0 0 0 -> xyz=0.128 0 0.04 rpy=0 0 0
- joint Joint_5: limit lower=-2.269 upper=2.269 effort=1 velocity=1 -> lower=-2.2689 upper=2.2689 effort=1 velocity=1; origin xyz=0.2955 0 0 rpy=0 0 0 -> xyz=0.297 0 0 rpy=0 0 0
- joint Joint_6: limit lower=-6.981 upper=6.981 effort=1 velocity=1 -> lower=-4.2237 upper=4.2237 effort=1 velocity=1

File: Assests/Robot APCC/IRB_1300_1400_URDF/urdf/IRB_1300_1400_URDF_with_fixture.urdf (robot description, URDF)
Before this commit: robot IRB-1300 1150 URDF, 7 links, 6 joints
Links:
- removed link Link1
- removed link Link2
- removed link Link3
- removed link Link4
- removed link Link5
- removed link Link6
- removed link base_link
- added link Base_link, mass 13.186356777892; collision mesh filename=../meshes/Base_link.STL; visual mesh filename=../meshes/Base_link.STL
- added link Link_1, mass 16.335535333141; collision mesh filename=../meshes/Link_1.STL; visual mesh filename=../meshes/Link_1.STL
- added link Link_2, mass 15.4420852413982; collision mesh filename=../meshes/Link_2.STL; visual mesh filename=../meshes/Link_2.STL
- added link Link_3, mass 4.42114015837963; collision mesh filename=../meshes/Link_3.STL; visual mesh filename=../meshes/Link_3.STL
- added link Link_4, mass 5.24616552302721; collision mesh filename=../meshes/Link_4.STL; visual mesh filename=../meshes/Link_4.STL
- added link Link_5, mass 0.604631449587936; collision mesh filename=../meshes/Link_5.STL; visual mesh filename=../meshes/Link_5.STL
- added link Link_6, mass 0.0169042353816242; collision mesh filename=../meshes/Link_7.STL; visual mesh filename=../meshes/Link_7.STL
- added link ee_link
Joints:
- removed joint Joint1
- removed joint Joint2
- removed joint Joint3
- removed joint Joint4
- removed joint Joint5
- removed joint Joint6
- added joint Joint_1: type revolute, parent Base_link, child Link_1, origin xyz=0 0 0.254 rpy=0 0 0, axis 0 0 1, limit lower=-3.1416 upper=3.1416 effort=1 velocity=1
- added joint Joint_2: type revolute, parent Link_1, child Link_2, origin xyz=0.15 0 0.29 rpy=0 0 0, axis 0 1 0, limit lower=-1.6581 upper=2.7053 effort=1 velocity=1
- added joint Joint_3: type revolute, parent Link_2, child Link_3, origin xyz=0 0 0.575 rpy=0 0 0, axis 0 1 0, limit lower=-3.6652 upper=1.2043 effort=1 velocity=1
- added joint Joint_4: type revolute, parent Link_3, child Link_4, origin xyz=0.1295 0 0.04 rpy=0 0 0, axis 1 0 0, limit lower=-4.0143 upper=4.0143 effort=1 velocity=1
- added joint Joint_5: type revolute, parent Link_4, child Link_5, origin xyz=0.5455 0 0 rpy=0 0 0, axis 0 1 0, limit lower=-2.2689 upper=2.2689 effort=1 velocity=1
- added joint Joint_6: type revolute, parent Link_5, child Link_6, origin xyz=0.092 0 0 rpy=0 1.5708 0, axis 0 0 1, limit lower=-6.9813 upper=6.9813 effort=1 velocity=1
- added joint ee_joint: type fixed, parent Link_6, child ee_link, origin xyz=0.0998237 0.123033 0.0828027 rpy=0.001199 0.000599 2.782547

File: Assests/Robot APCC/IRB_1300_900_URDF/IRB-1300-900 URDF_v2/urdf/IRB_1300_900_URDF.urdf (robot description, URDF)
Before this commit: robot IRB-1300 1400 URDF, 7 links, 6 joints
Links:
- removed link Base
- added link Base_link, mass 13191690802.2938; collision mesh filename=../meshes/Base_link.STL; visual mesh filename=../meshes/Base_link.STL
- link Link_1: mass 16.335535333141 -> 15143711685.0337
- link Link_2: mass 15.4420852413982 -> 13168240511.6789
- link Link_3: mass 4.42114015837963 -> 4421135022.18643
- link Link_4: mass 5.24616552302721 -> 3695342210.06587
- link Link_5: mass 0.604631449587936 -> 586394466.626242
- link Link_6: mass 0.0169042353816242 -> 7900320.12561475; geometry collision mesh filename=../meshes/Link_6.STL; visual mesh filename=../meshes/Link_6.STL
Joints:
- joint Joint_1: limit lower=-3.1416 upper=3.1416 effort=1 velocity=1 -> lower=-3.142 upper=3.142 effort=1 velocity=1; parent Base -> Base_link
- joint Joint_2: limit lower=-1.6581 upper=2.7053 effort=1 velocity=1 -> lower=-1.745 upper=2.269 effort=1 velocity=1; origin xyz=0.15 0 0.29 rpy=0 0 0 -> xyz=0.05 0 0.29 rpy=0 0 0
- joint Joint_3: limit lower=-3.6652 upper=1.2043 effort=1 velocity=1 -> lower=-3.665 upper=1.134 effort=1 velocity=1; origin xyz=0 0 0.575 rpy=0 0 0 -> xyz=0 0 0.425 rpy=0 0 0
- joint Joint_4: limit lower=-4.0143 upper=4.0143 effort=1 velocity=1 -> lower=-4.014 upper=4.014 effort=1 velocity=1
- joint Joint_5: limit lower=-2.2689 upper=2.2689 effort=1 velocity=1 -> lower=-2.269 upper=2.269 effort=1 velocity=1; origin xyz=0.5455 0 0 rpy=0 0 0 -> xyz=0.2955 0 0 rpy=0 0 0
- joint Joint_6: limit lower=-6.9813 upper=6.9813 effort=1 velocity=1 -> lower=-6.981 upper=6.981 effort=1 velocity=1; origin xyz=0.092 0 0 rpy=0 1.5708 0 -> xyz=0.09 0 0 rpy=0 1.5708 0

File: Assests/Robot APCC/IRB_1300_900_URDF/IRB-1300-900 URDF_v2/urdf/IRB_1300_900_URDF_with_fixture.urdf (robot description, URDF)
Before this commit: robot IRB-1300 1400 URDF, 8 links, 7 joints
Links:
- removed link Base
- added link Base_link, mass 13191690802.2938; collision mesh filename=../meshes/Base_link.STL; visual mesh filename=../meshes/Base_link.STL
- link Link_1: mass 16.335535333141 -> 15143711685.0337
- link Link_2: mass 15.4420852413982 -> 13168240511.6789
- link Link_3: mass 4.42114015837963 -> 4421135022.18643
- link Link_4: mass 5.24616552302721 -> 3695342210.06587
- link Link_5: mass 0.604631449587936 -> 586394466.626242
- link Link_6: mass 0.0169042353816242 -> 7900320.12561475; geometry collision mesh filename=../meshes/Link_6.STL; visual mesh filename=../meshes/Link_6.STL
Joints:
- joint Joint_1: limit lower=-3.1416 upper=3.1416 effort=1 velocity=1 -> lower=-3.142 upper=3.142 effort=1 velocity=1; parent Base -> Base_link
- joint Joint_2: limit lower=-1.6581 upper=2.7053 effort=1 velocity=1 -> lower=-1.745 upper=2.269 effort=1 velocity=1; origin xyz=0.15 0 0.29 rpy=0 0 0 -> xyz=0.05 0 0.29 rpy=0 0 0
- joint Joint_3: limit lower=-3.6652 upper=1.2043 effort=1 velocity=1 -> lower=-3.665 upper=1.134 effort=1 velocity=1; origin xyz=0 0 0.575 rpy=0 0 0 -> xyz=0 0 0.425 rpy=0 0 0
- joint Joint_4: limit lower=-4.0143 upper=4.0143 effort=1 velocity=1 -> lower=-4.014 upper=4.014 effort=1 velocity=1
- joint Joint_5: limit lower=-2.2689 upper=2.2689 effort=1 velocity=1 -> lower=-2.269 upper=2.269 effort=1 velocity=1; origin xyz=0.5455 0 0 rpy=0 0 0 -> xyz=0.2955 0 0 rpy=0 0 0
- joint Joint_6: limit lower=-6.9813 upper=6.9813 effort=1 velocity=1 -> lower=-6.981 upper=6.981 effort=1 velocity=1; origin xyz=0.092 0 0 rpy=0 1.5708 0 -> xyz=0.09 0 0 rpy=0 1.5708 0
